Commit message: Add script to classify object with CNN

File: project_robot_description/urdf/sensors/xtion_pro_live.urdf.xacro (robot description, xacro)
@@ -1,5 +1,5 @@
 <?xml version="1.0"?>
 <robot xmlns:xacro="http://ros.org/wiki/xacro">
-  <xacro:include filename="$(find mastering_ros_robot_description_pkg)/urdf/sensors/xtion_pro_live.gazebo.xacro"/>
+  <xacro:include filename="$(find project_robot_description)/urdf/sensors/xtion_pro_live.gazebo.xacro"/>
   <xacro:macro name="dummy_inertial">
     <inertial>
@@ -37,5 +37,5 @@
       <collision>
       <geometry>
-          <mesh filename="package://mastering_ros_robot_description_pkg/meshes/sensors/xtion_pro_live/xtion_pro_live.dae"/>
+          <mesh filename="package://project_robot_description/meshes/sensors/xtion_pro_live/xtion_pro_live.dae"/>
       </geometry>
       </collision>
