Commit message: fix camera

File: project_robot_description/urdf/seven_dof_arm.xacro (robot description, xacro)
@@ -1,4 +1,5 @@
 <?xml version="1.0"?>
 <robot name="seven_dof_arm" xmlns:xacro="http://ros.org/wiki/xacro">
+  <xacro:include filename="$(find project_robot_description)/urdf/seven_dof_arm.gazebo"/>
   <!-- Include materials -->
     <material name="Black">
@@ -400,5 +401,5 @@
       <origin xyz="0.08 0 0" rpy="0 0 0"/>
     </joint>
-    <link name="camera">
+    <link name="camera_link">
       <collision>
         <origin xyz="0 0 0" rpy="0 0 0"/>
@@ -425,5 +426,5 @@
       <origin xyz=".2 0 0" rpy="0 0 0"/>
       <parent link="wrist_pitch_link"/>
-      <child link="camera"/>
+      <child link="camera_link"/>
     </joint>
   <xacro:include filename="$(find mastering_ros_robot_description_pkg)/urdf/sensors/xtion_pro_live.urdf.xacro"/>

Commit message: configure the launch file to open a custom world

File: project_robot_description/urdf/seven_dof_arm.xacro (robot description, xacro)
@@ -424,6 +424,6 @@
     <joint name="camera_joint" type="fixed">
       <axis xyz="0 1 0" />
-      <origin xyz=".2 0 0" rpy="0 0 0"/>
-      <parent link="wrist_pitch_link"/>
+      <origin xyz=".1 0 0" rpy="0 0 0"/>
+      <parent link="base_link"/>
       <child link="camera_link"/>
     </joint>

Commit message: Fix gripper + gazebo_grasp_plugin

File: project_robot_description/urdf/seven_dof_arm.xacro (robot description, xacro)
@@ -116,5 +116,5 @@
       </geometry>
       </collision>>
-	<xacro:inertial_matrix mass="1"/>
+	<xacro:inertial_matrix mass="1000"/>
   </link>
   <gazebo reference="base_link">
@@ -348,4 +348,10 @@
       <material name="White" />
     </visual>
+    <collision>
+      <origin xyz="0.04 -0.03 0"/>
+      <geometry>
+        <box size="${left_gripper_len} ${left_gripper_width} ${left_gripper_height}" />
+      </geometry>
+    </collision>
 	<xacro:inertial_matrix mass="1"/>
   </link>
@@ -373,4 +379,10 @@
       <material name="White" />
     </visual>
+    <collision>
+      <origin xyz="0.04 0.03 0"/>
+      <geometry>
+        <box size="${right_gripper_len} ${right_gripper_width} ${right_gripper_height}" />
+      </geometry>
+    </collision>
 	<xacro:inertial_matrix mass="1"/>
   </link>
@@ -413,5 +425,5 @@
           <box size="${cameraSize} ${cameraSize} ${cameraSize}"/>
         </geometry>
-        <material name="green"/>
+        <material name="Black"/>
       </visual>
       <inertial>
@@ -424,9 +436,9 @@
     <joint name="camera_joint" type="fixed">
       <axis xyz="0 1 0" />
-      <origin xyz=".1 0 0" rpy="0 0 0"/>
+      <origin xyz=".04 0 0" rpy="0 0 0"/>
       <parent link="base_link"/>
       <child link="camera_link"/>
     </joint>
-  <xacro:include filename="$(find mastering_ros_robot_description_pkg)/urdf/sensors/xtion_pro_live.urdf.xacro"/>
+  <xacro:include filename="$(find project_robot_description)/urdf/sensors/xtion_pro_live.urdf.xacro"/>
 <!-- ///////////////////////////////////////////////////////////////////////////////////////////////////////////////////// -->
   <!-- Transmissions for ROS Control -->
@@ -446,3 +458,20 @@
     </plugin>
   </gazebo>
+  <gazebo>
+  <plugin name="gazebo_grasp_fix" filename="libgazebo_grasp_fix.so">
+    <arm>
+      <arm_name>seven_dof_arm</arm_name>
+      <palm_link>gripper_roll_link</palm_link>
+      <gripper_link>gripper_finger_link1</gripper_link>
+      <gripper_link>gripper_finger_link2</gripper_link>
+    </arm>
+    <forces_angle_tolerance>100</forces_angle_tolerance>
+    <update_rate>4</update_rate>
+    <grip_count_threshold>4</grip_count_threshold>
+    <max_grip_count>8</max_grip_count>
+    <release_tolerance>0.005</release_tolerance>
+    <disable_collisions_on_attach>false</disable_collisions_on_attach>
+    <contact_topic>__default_topic__</contact_topic>
+  </plugin>
+  </gazebo>
 </robot>

Commit message: Fix robot slipping on the ground plane

File: project_robot_description/urdf/seven_dof_arm.xacro (robot description, xacro)
@@ -75,34 +75,11 @@
 <!-- BOTTOM FIXED LINK
 This link is the base of the arm in which arm is placed
--->
-<!-- ///////////////////////////////////////////////////////////////////////////////////////////////////////////////////// -->
-  <joint name="bottom_joint" type="fixed">
-    <origin xyz="0 0 0" rpy="0 0 0" />
-    <parent link="base_link"/>
-    <child link="bottom_link"/>
-  </joint>
-  <link name="bottom_link">
-    <visual>
-      <origin xyz=" 0 0 -0.04"  rpy="0 0 0"/>
-      <geometry>
-	       <box size="1 1 0.02" />
-      </geometry>
-      <material name="Brown" />
-    </visual>
-    <collision>
-      <origin xyz=" 0 0 -0.04"  rpy="0 0 0"/>
-      <geometry>
-	       <box size="1 1 0.02" />
-      </geometry>
-      </collision>>
-  </link>
-  <gazebo reference="bottom_link">
-    <material>Gazebo/White</material>
-  </gazebo>
+--> <link name="world" />
+<!-- ///////////////////////////////////////////////////////////////////////////////////////////////////////////////////// -->
 <!-- ///////////////////////////////////////////////////////////////////////////////////////////////////////////////////// -->
   <!-- BASE LINK -->
   <link name="base_link">
     <visual>
-      <origin xyz="0 0 0" rpy="${M_PI/2} 0 0" /> <!-- rotate PI/2 -->
+      <origin xyz="0 0 0" rpy="0 0 0" /> <!-- rotate PI/2 -->
       <geometry>
 	       <box size="0.1 0.1 0.1" />
@@ -111,14 +88,22 @@
     </visual>
     <collision>
-      <origin xyz="0 0 0" rpy="${M_PI/2} 0 0" /> <!-- rotate PI/2 -->
+      <origin xyz="0 0 0" rpy="0 0 0" /> <!-- rotate PI/2 -->
       <geometry>
 	       <box size="0.1 0.1 0.1" />
       </geometry>
-      </collision>>
-	<xacro:inertial_matrix mass="1000"/>
+      </collision>
+        <inertial>
+            <mass value="0.1" />
+            <inertia ixx="0.03" iyy="0.03" izz="0.03" ixy="0.0" ixz="0.0" iyz="0.0" />
+        </inertial>
   </link>
   <gazebo reference="base_link">
     <material>Gazebo/White</material>
-  </gazebo>
+    <turnGravityOff>false</turnGravityOff>
+  </gazebo>
+   <joint name="bottom_joint" type="fixed">
+    <parent link="world"/>
+    <child link="base_link"/>
+  </joint>
   <joint name="shoulder_pan_joint" type="revolute">
     <parent link="base_link"/>
